Commit message: a working phase2

File: ros2_ws/src/alicia_d_ros2_upstream/alicia_d_descriptions/urdf/Alicia_D_v5_6/Alicia_D_v5_6_gripper_50mm.urdf (robot description, URDF)
Before this commit: robot Alicia_D_v5_6_gripper_50mm, 10 links, 9 joints
Joints:
- joint Joint1: origin xyz=0 0 0.1295 rpy=0 -0.0397818431857344 0 -> xyz=${0.0 + joint_origin_xyz_corrections['Joint1'][0]} ${0.0 + joint_origin_xyz_corrections['Joint1'][1]} ${0.1295 + joint_origin_xyz_corrections['Joint1'][2]} rpy=${0.0 + joint_origin_rpy_corrections['Joint1'][0] * pi / 180.0} ${-0.0397818431857344 + joint_origin_rpy_corrections['Joint1'][1] * pi / 180.0} ${0.0 + joint_origin_rpy_corrections['Joint1'][2] * pi / 180.0}
- joint Joint2: origin xyz=0.00170499781414124 0 0.0428360815487805 rpy=1.5707963267949 -1.5707963267949 0 -> xyz=${0.00170499781414124 + joint_origin_xyz_corrections['Joint2'][0]} ${0.0 + joint_origin_xyz_corrections['Joint2'][1]} ${0.0428360815487805 + joint_origin_xyz_corrections['Joint2'][2]} rpy=${1.5707963267949 + joint_origin_rpy_corrections['Joint2'][0] * pi / 180.0} ${-1.5707963267949 + joint_origin_rpy_corrections['Joint2'][1] * pi / 180.0} ${0.0 + joint_origin_rpy_corrections['Joint2'][2] * pi / 180.0}
- joint Joint3: origin xyz=0.223671302741224 0.0226916129580064 -4.99999999962493E-05 rpy=0 0 -2.35619449019234 -> xyz=${0.223671302741224 + joint_origin_xyz_corrections['Joint3'][0]} ${0.0226916129580064 + joint_origin_xyz_corrections['Joint3'][1]} ${-4.99999999962493E-05 + joint_origin_xyz_corrections['Joint3'][2]} rpy=${0.0 + joint_origin_rpy_corrections['Joint3'][0] * pi / 180.0} ${0.0 + joint_origin_rpy_corrections['Joint3'][1] * pi / 180.0} ${-2.35619449019234 + joint_origin_rpy_corrections['Joint3'][2] * pi / 180.0}
- joint Joint4: origin xyz=0.00211000000000178 -0.0990000000000033 -0.0002000000000025 rpy=1.5707963267949 0 0 -> xyz=${0.00211000000000178 + joint_origin_xyz_corrections['Joint4'][0]} ${-0.0990000000000033 + joint_origin_xyz_corrections['Joint4'][1]} ${-0.0002000000000025 + joint_origin_xyz_corrections['Joint4'][2]} rpy=${1.5707963267949 + joint_origin_rpy_corrections['Joint4'][0] * pi / 180.0} ${0.0 + joint_origin_rpy_corrections['Joint4'][1] * pi / 180.0} ${0.0 + joint_origin_rpy_corrections['Joint4'][2] * pi / 180.0}
- joint Joint5: origin xyz=0 -0.000500000000001193 0.12235 rpy=1.5707963267949 0 0 -> xyz=${0.0 + joint_origin_xyz_corrections['Joint5'][0]} ${-0.000500000000001193 + joint_origin_xyz_corrections['Joint5'][1]} ${0.12235 + joint_origin_xyz_corrections['Joint5'][2]} rpy=${1.5707963267949 + joint_origin_rpy_corrections['Joint5'][0] * pi / 180.0} ${0.0 + joint_origin_rpy_corrections['Joint5'][1] * pi / 180.0} ${0.0 + joint_origin_rpy_corrections['Joint5'][2] * pi / 180.0}
- joint Joint6: origin xyz=-0.00384999999999935 0.0574999999999998 -0.00100000000000219 rpy=-1.5707963267949 0 0 -> xyz=${-0.00384999999999935 + joint_origin_xyz_corrections['Joint6'][0]} ${0.0574999999999998 + joint_origin_xyz_corrections['Joint6'][1]} ${-0.00100000000000219 + joint_origin_xyz_corrections['Joint6'][2]} rpy=${-1.5707963267949 + joint_origin_rpy_corrections['Joint6'][0] * pi / 180.0} ${0.0 + joint_origin_rpy_corrections['Joint6'][1] * pi / 180.0} ${0.0 + joint_origin_rpy_corrections['Joint6'][2] * pi / 180.0}

File: ros2_ws/src/alicia_d_ros2_upstream/alicia_d_moveit/config/Alicia_D_v5_6_gripper_50mm.urdf.xacro (robot description, xacro)
@@ -5,6 +5,21 @@
     <xacro:arg name="hw_gripper_type" default="50mm" />
     <xacro:arg name="hw_default_speed_deg_s" default="20.0" />
+    <xacro:arg name="kinematic_calibration_file" default="$(find alicia_d_moveit)/config/kinematic_calibration.yaml" />
+    <xacro:property name="kinematic_calibration_file_path" value="$(arg kinematic_calibration_file)" />
+    <xacro:property name="kinematic_calibration" value="${xacro.load_yaml(kinematic_calibration_file_path)}" />
+    <xacro:property name="joint_offsets" value="${kinematic_calibration['joint_position_offsets_rad']}" />
+    <xacro:property name="joint_origin_xyz_corrections" value="${kinematic_calibration['joint_origin_xyz_corrections_m']}" />
+    <xacro:property name="joint_origin_rpy_corrections" value="${kinematic_calibration['joint_origin_rpy_corrections_deg']}" />
+    <xacro:property name="tcp_correction" value="${kinematic_calibration['tcp_correction']}" />
     <!-- Import alicia_d_descriptions urdf file for v5_6 50mm -->
     <xacro:include filename="$(find alicia_d_descriptions)/urdf/Alicia_D_v5_6/Alicia_D_v5_6_gripper_50mm.urdf" />
+    <link name="tool0" />
+    <joint name="tool0_fixed" type="fixed">
+        <parent link="gripper_center" />
+        <child link="tool0" />
+        <origin
+            xyz="${tcp_correction['xyz'][0]} ${tcp_correction['xyz'][1]} ${tcp_correction['xyz'][2]}"
+            rpy="${tcp_correction['rpy_deg'][0] * pi / 180.0} ${tcp_correction['rpy_deg'][1] * pi / 180.0} ${tcp_correction['rpy_deg'][2] * pi / 180.0}" />
+    </joint>
     <!-- Import control_xacro -->
     <xacro:include filename="alicia_d_descriptions.ros2_control.xacro" />
@@ -15,4 +30,5 @@
         hw_port="$(arg hw_port)"
         hw_gripper_type="$(arg hw_gripper_type)"
-        hw_default_speed_deg_s="$(arg hw_default_speed_deg_s)"/>
+        hw_default_speed_deg_s="$(arg hw_default_speed_deg_s)"
+        hw_joint_position_offsets_rad="${joint_offsets['Joint1']},${joint_offsets['Joint2']},${joint_offsets['Joint3']},${joint_offsets['Joint4']},${joint_offsets['Joint5']},${joint_offsets['Joint6']}"/>
 </robot>

File: ros2_ws/src/alicia_d_ros2_upstream/alicia_d_moveit/config/Alicia_D_v5_6_gripper_50mm_demo.urdf.xacro (robot description, xacro)
@@ -2,6 +2,20 @@
 <robot xmlns:xacro="http://www.ros.org/wiki/xacro" name="Alicia_D_v5_6_gripper_50mm">
     <xacro:arg name="initial_positions_file" default="initial_positions.yaml" />
+    <xacro:arg name="kinematic_calibration_file" default="$(find alicia_d_moveit)/config/kinematic_calibration.yaml" />
+    <xacro:property name="kinematic_calibration_file_path" value="$(arg kinematic_calibration_file)" />
+    <xacro:property name="kinematic_calibration" value="${xacro.load_yaml(kinematic_calibration_file_path)}" />
+    <xacro:property name="joint_origin_xyz_corrections" value="${kinematic_calibration['joint_origin_xyz_corrections_m']}" />
+    <xacro:property name="joint_origin_rpy_corrections" value="${kinematic_calibration['joint_origin_rpy_corrections_deg']}" />
+    <xacro:property name="tcp_correction" value="${kinematic_calibration['tcp_correction']}" />
     <!-- Import alicia_d_descriptions urdf file for v5_6 50mm -->
     <xacro:include filename="$(find alicia_d_descriptions)/urdf/Alicia_D_v5_6/Alicia_D_v5_6_gripper_50mm.urdf" />
+    <link name="tool0" />
+    <joint name="tool0_fixed" type="fixed">
+        <parent link="gripper_center" />
+        <child link="tool0" />
+        <origin
+            xyz="${tcp_correction['xyz'][0]} ${tcp_correction['xyz'][1]} ${tcp_correction['xyz'][2]}"
+            rpy="${tcp_correction['rpy_deg'][0] * pi / 180.0} ${tcp_correction['rpy_deg'][1] * pi / 180.0} ${tcp_correction['rpy_deg'][2] * pi / 180.0}" />
+    </joint>
     <!-- Import fake control_xacro for demo mode -->
     <xacro:include filename="alicia_d_descriptions.ros2_control.fake.xacro" />

File: ros2_ws/src/alicia_d_ros2_upstream/alicia_d_moveit/config/alicia_d_descriptions.ros2_control.xacro (robot description, xacro)
@@ -5,5 +5,6 @@
                  hw_debug_mode:=false
                  hw_gripper_type:=50mm
-                 hw_default_speed_deg_s:=20.0">
+                 hw_default_speed_deg_s:=20.0
+                 hw_joint_position_offsets_rad:=0,0,0,0,0,0">
         <xacro:property name="initial_positions" value="${xacro.load_yaml(initial_positions_file)['initial_positions']}"/>
         <ros2_control name="${name}" type="system">
@@ -13,4 +14,5 @@
                 <param name="gripper_type">${hw_gripper_type}</param>
                 <param name="default_speed_deg_s">${hw_default_speed_deg_s}</param>
+                <param name="joint_position_offsets_rad">${hw_joint_position_offsets_rad}</param>
             </hardware>
             <joint name="Joint1">
